File: mcu.kicad_sch (KiCad schematic)
At the start: 29 parts, among them U1 nRF5340-QKxx

Commit message: added W5100
Parts:
- C1: renamed from C?; footprint (none) -> Connector_RJ:RJ45_Cetus_J1B1211CCD_Horizontal
- C10: renamed from C?; value C -> 100n
- R1: renamed from R?; value R -> 2R2
- R2: renamed from R?; value R -> 10k
- gave numbers to parts that had none: 24
Connections:
- net GND: now also C15.2, C16.2, C17.2, C18.2, C19.2, C2.2, C20.2, C21.2, C22.2, C7.2
- net VDD: now also C15.1, C16.1, C17.1, C18.1, C19.1, C2.1, C20.1, C21.1, C22.1, C7.1
- net NFC2: now reaches U1.AA1 (NFC2/P0.03)
- net D+: now reaches U1.B2 (D+)
- net D-: now reaches U1.B4 (D-)
- net NFC1: now reaches U1.W1 (NFC1/P0.02)
Other:
- moved on the sheet: C1, C10, C11, C12, C13, C14, C15, C16, C17, C18, C19, C2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

Commit message: Finishe PoE and ethernet
Parts:
- removed C1: 4u7, Connector_RJ:RJ45_Cetus_J1B1211CCD_Horizontal, symbol Device:C
- removed C10, C15, C16, C17, C18, C19, C20, C21, C22, C8: 100n, symbol Device:C
- removed C11: 2n2, symbol Device:C
- removed C12, C14, C2, C6, C7: 1u, symbol Device:C
- removed C13: 0p7, symbol Device:C
- removed C3: 4u7, symbol Device:C
- removed C4, C9: 10p, symbol Device:C
- removed C5: DNP, symbol Device:C
- removed L1, L3: 10u, symbol Device:L
- removed L2: 2n2, symbol Device:L
- removed R1: 2R2, symbol Device:R
- removed R2: 10k, symbol Device:R
- removed U1: nRF5340-QKxx, Package_DFN_QFN:Nordic_AQFN-94-1EP_7x7mm_P0.4mm, symbol MCU_Nordic:nRF5340-QKxx
- removed Y1: 32MHz, Crystal:Crystal_SMD_3225-4Pin_3.2x2.5mm, symbol Device:Crystal_GND24
- added C? (x5): 1u, symbol Device:C
- added C?: DNP, symbol Device:C
- added C? (x10): 100n, symbol Device:C
- added C?: 4u7, symbol Device:C
- added C?: 4u7, Connector_RJ:RJ45_Cetus_J1B1211CCD_Horizontal, symbol Device:C
- added C? (x2): 10p, symbol Device:C
- added C?: 2n2, symbol Device:C
- added C?: 0p7, symbol Device:C
- added L? (x2): 10u, symbol Device:L
- added L?: 2n2, symbol Device:L
- added R?: 10k, symbol Device:R
- added R?: 2R2, symbol Device:R
- added U?: nRF5340-QKxx, Package_DFN_QFN:Nordic_AQFN-94-1EP_7x7mm_P0.4mm, symbol MCU_Nordic:nRF5340-QKxx
- added Y?: 32MHz, Crystal:Crystal_SMD_3225-4Pin_3.2x2.5mm, symbol Device:Crystal_GND24
Connections:
- net D+: now also U?.B2 (D+)
- net D-: now also U?.B4 (D-)
- net GND: now also C?.2, C?.2, C?.2, C?.2, C?.2, C?.2, C?.2, C?.2, C?.2, C?.2, C?.2, C?.2, C?.2, C?.2, C?.2, C?.2, C?.2, C?.2, C?.2, C?.2, C?.2, C?.2, U?.EP (VSS), Y?.2, Y?.4
- net NFC1: now also U?.W1 (NFC1/P0.02)
- net NFC2: now also U?.AA1 (NFC2/P0.03)
- net VBUS: now also R?.1
- net VDD: now also C?.1, C?.1, C?.1, C?.1, C?.1, C?.1, C?.1, C?.1, C?.1, C?.1, R?.1, U?.A19 (VDD), U?.AC1 (VDD), U?.AG1 (VDD), U?.AJ31 (VDD), U?.AL11 (VDD), U?.AL17 (VDD), U?.AL25 (VDD), U?.AL3 (VDD), U?.AL7 (VDD), U?.B28 (VDD), U?.B8 (VDD), U?.C1 (VDD), U?.E1 (VDDH), U?.E31 (VDD), U?.L1 (VDD), U?.N31 (VDD), U?.U1 (VDD)
- new net: C?.1, C?.1, L?.1, U?.A27 (DECR), U?.G31 (DECRF)
- new net: L?.2, U?.A21 (DCC)
- new net: C?.1, U?.A13 (DECA)
- new net: C?.1, L?.1
- new net: C?.1, U?.A23 (DECN)
- new net: C?.1, U?.B6 (DECUSB)
- new net: C?.1, L?.1, U?.A15 (DECD)
- new net: C?.1, R?.2, U?.A5 (VBUS)
- new net: C?.1, U?.B30 (XC2), Y?.1
- new net: C?.1, R?.2, U?.AC31 (~{RESET})
- new net: C?.1, U?.C31 (XC1), Y?.3
- new net: L?.2, U?.B10 (DCCD)
- new net: C?.1, L?.2, U?.L31 (ANT)

Commit message: Added USB port
Parts:
- removed C? (x5): 1u, symbol Device:C
- removed C?: DNP, symbol Device:C
- removed C? (x10): 100n, symbol Device:C
- removed C?: 4u7, symbol Device:C
- removed C?: 4u7, Connector_RJ:RJ45_Cetus_J1B1211CCD_Horizontal, symbol Device:C
- removed C? (x2): 10p, symbol Device:C
- removed C?: 2n2, symbol Device:C
- removed C?: 0p7, symbol Device:C
- removed L? (x2): 10u, symbol Device:L
- removed L?: 2n2, symbol Device:L
- removed R?: 10k, symbol Device:R
- removed R?: 2R2, symbol Device:R
- removed U?: nRF5340-QKxx, Package_DFN_QFN:Nordic_AQFN-94-1EP_7x7mm_P0.4mm, symbol MCU_Nordic:nRF5340-QKxx
- removed Y?: 32MHz, Crystal:Crystal_SMD_3225-4Pin_3.2x2.5mm, symbol Device:Crystal_GND24
Connections:
- no-connect marks 1 -> 0
