File: W5100_PoE.kicad_sch (KiCad schematic)
At the start: 82 parts, among them J2 ARJM11C7-114-BA-EW2, T1 FA2805, U10 USBLC6-2SC6, U11 USBLC6-2SC6, U3 W5100S, U4 TLV431DBZ, U5 VO618A, U6 SI3402, U8 VO618A, Y2 25MHz

Commit message: Routing almost done
Parts:
- C26: value 470u -> 220u; footprint Capacitor_Tantalum_SMD:CP_EIA-2012-12_Kemet-R -> Capacitor_SMD:CP_Elec_5x5.3
Connections:
- net GND: now also U3.49 (GND)
- net at D6.1 (K), T1.2, U6.18 (SWO): no longer C29.2
- net Earth: now reaches C45.2, C49.2, C51.2, C55.2, R16.2, U6.21 (VNEG), U6.9 (VNEG)
- net Earth: now also C29.2
Changed lines of the file:
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@@
   (junction (at 214.63 222.25) (diameter 0) (color 0 0 0 0)
   )
-  (junction (at 135.89 63.5) (diameter 0) (color 0 0 0 0)
-  )
   (junction (at 135.89 81.28) (diameter 0) (color 0 0 0 0)
   )
@@
   (junction (at 293.37 144.78) (diameter 0) (color 0 0 0 0)
   )
+  (junction (at 241.3 86.36) (diameter 0) (color 0 0 0 0)
+  )
   (junction (at 284.48 55.88) (diameter 0) (color 0 0 0 0)
   )
@@
   (junction (at 122.555 254.635) (diameter 0) (color 0 0 0 0)
   )
-  (junction (at 80.01 68.58) (diameter 0) (color 0 0 0 0)
-  )
   (junction (at 201.93 250.19) (diameter 0) (color 0 0 0 0)
   )
@@
     (stroke (width 0) (type default) (color 0 0 0 0))
   )
+  (wire (pts (xy 121.92 68.58) (xy 115.57 68.58))
+    (stroke (width 0) (type default) (color 0 0 0 0))
+  )
   (wire (pts (xy 323.85 105.41) (xy 326.39 105.41))
     (stroke (width 0) (type default) (color 0 0 0 0))
@@
     (stroke (width 0) (type default) (color 0 0 0 0))
   )
-  (wire (pts (xy 80.01 69.85) (xy 80.01 68.58))
+  (wire (pts (xy 80.01 57.15) (xy 80.01 62.23))
     (stroke (width 0) (type default) (color 0 0 0 0))
   )
@@
     (stroke (width 0) (type default) (color 0 0 0 0))
   )
+  (wire (pts (xy 115.57 68.58) (xy 115.57 69.85))
+    (stroke (width 0) (type default) (color 0 0 0 0))
+  )
   (wire (pts (xy 68.58 96.52) (xy 78.74 96.52))
     (stroke (width 0) (type default) (color 0 0 0 0))
@@
     (stroke (width 0) (type default) (color 0 0 0 0))
   )
-  (wire (pts (xy 135.89 35.56) (xy 135.89 40.64))
+  (wire (pts (xy 241.3 86.36) (xy 241.3 87.63))
     (stroke (width 0) (type default) (color 0 0 0 0))
   )
-  (wire (pts (xy 135.89 68.58) (xy 135.89 63.5))
+  (wire (pts (xy 135.89 35.56) (xy 135.89 40.64))
     (stroke (width 0) (type default) (color 0 0 0 0))
   )
@@
     (stroke (width 0) (type default) (color 0 0 0 0))
   )
-  (wire (pts (xy 80.01 57.15) (xy 80.01 68.58))
-    (stroke (width 0) (type default) (color 0 0 0 0))
-  )
   (wire (pts (xy 231.14 176.53) (xy 236.22 176.53))
     (stroke (width 0) (type default) (color 0 0 0 0))
@@
     (stroke (width 0) (type default) (color 0 0 0 0))
   )
-  (wire (pts (xy 270.51 144.78) (xy 270.51 166.37))
+  (wire (pts (xy 135.89 68.58) (xy 135.89 69.85))
     (stroke (width 0) (type default) (color 0 0 0 0))
   )
-  (wire (pts (xy 80.01 68.58) (xy 121.92 68.58))
+  (wire (pts (xy 270.51 144.78) (xy 270.51 166.37))
     (stroke (width 0) (type default) (color 0 0 0 0))
   )
@@
     (pin "2")
   )
+  (symbol (lib_id "power:GND") (at 115.57 69.85 0) (unit 1)
+    (in_bom yes) (on_board yes)
+    (property "Reference" "#PWR0154" (id 0) (at 115.57 76.2 0)
+      (effects (font (size 1.27 1.27)) hide)
+    )
+    (property "Value" "GND" (id 1) (at 115.57 73.66 0))
+    (property "Footprint" "" (id 2) (at 115.57 69.85 0)
+      (effects (font (size 1.27 1.27)) hide)
+    )
+    (property "Datasheet" "" (id 3) (at 115.57 69.85 0)
+      (effects (font (size 1.27 1.27)) hide)
+    )
+    (pin "1")
+  )
   (symbol (lib_id "Device:C") (at 293.37 80.01 0) (unit 1)
     (in_bom yes) (on_board yes)
@@
     (pin "2")
   )
+  (symbol (lib_id "power:Earth") (at 135.89 69.85 0) (unit 1)
+    (in_bom yes) (on_board yes) (fields_autoplaced)
+    (property "Reference" "#PWR0155" (id 0) (at 135.89 76.2 0)
+      (effects (font (size 1.27 1.27)) hide)
+    )
+    (property "Value" "Earth" (id 1) (at 135.89 73.66 0)
+      (effects (font (size 1.27 1.27)) hide)
+    )
+    (property "Footprint" "" (id 2) (at 135.89 69.85 0)
+      (effects (font (size 1.27 1.27)) hide)
+    )
+    (property "Datasheet" "~" (id 3) (at 135.89 69.85 0)
+      (effects (font (size 1.27 1.27)) hide)
+    )
+    (pin "1")
+  )
   (symbol (lib_id "Device:R") (at 142.24 93.98 90) (unit 1)
     (in_bom yes) (on_board yes)
@@
       (effects (font (size 1.27 1.27)) (justify left))
     )
-    (property "Value" "470u" (id 1) (at 71.12 53.34 0)
+    (property "Value" "220u" (id 1) (at 71.12 53.34 0)
       (effects (font (size 1.27 1.27)) (justify left))
     )
-    (property "Footprint" "Capacitor_Tantalum_SMD:CP_EIA-2012-12_Kemet-R" (id 2) (at 80.9752 55.88 0)
+    (property "Footprint" "Capacitor_SMD:CP_Elec_5x5.3" (id 2) (at 80.9752 55.88 0)
       (effects (font (size 1.27 1.27)) hide)
     )
@@
     (pin "1")
   )
+  (symbol (lib_id "power:Earth") (at 241.3 87.63 0) (unit 1)
+    (in_bom yes) (on_board yes) (fields_autoplaced)
+    (property "Reference" "#PWR0153" (id 0) (at 241.3 93.98 0)
+      (effects (font (size 1.27 1.27)) hide)
+    )
+    (property "Value" "Earth" (id 1) (at 241.3 91.44 0)
+      (effects (font (size 1.27 1.27)) hide)
+    )
+    (property "Footprint" "" (id 2) (at 241.3 87.63 0)
+      (effects (font (size 1.27 1.27)) hide)
+    )
+    (property "Datasheet" "~" (id 3) (at 241.3 87.63 0)
+      (effects (font (size 1.27 1.27)) hide)
+    )
+    (pin "1")
+  )
   (symbol (lib_id "Device:R") (at 110.49 39.37 90) (unit 1)
     (in_bom yes) (on_board yes)
@@
     (pin "2")
   )
-  (symbol (lib_id "power:GND") (at 80.01 69.85 0) (unit 1)
+  (symbol (lib_id "power:GND") (at 80.01 62.23 0) (unit 1)
     (in_bom yes) (on_board yes)
-    (property "Reference" "#PWR0130" (id 0) (at 80.01 76.2 0)
+    (property "Reference" "#PWR0130" (id 0) (at 80.01 68.58 0)
       (effects (font (size 1.27 1.27)) hide)
     )
-    (property "Value" "GND" (id 1) (at 80.01 73.66 0))
-    (property "Footprint" "" (id 2) (at 80.01 69.85 0)
+    (property "Value" "GND" (id 1) (at 80.01 66.04 0))
+    (property "Footprint" "" (id 2) (at 80.01 62.23 0)
       (effects (font (size 1.27 1.27)) hide)
     )
-    (property "Datasheet" "" (id 3) (at 80.01 69.85 0)
+    (property "Datasheet" "" (id 3) (at 80.01 62.23 0)
       (effects (font (size 1.27 1.27)) hide)
     )
@@
     (pin "47")
     (pin "48")
+    (pin "49")
     (pin "5")
     (pin "6")

Commit message: Routing done
Changed lines of the file:
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@@
-    (effects (font (size 1.27 1.27)) (justify left bottom))
-  )
-  (label "CON_RD+" (at 411.48 132.08 0)
     (effects (font (size 1.27 1.27)) (justify left bottom))
   )
