File: _autosave-W5100_PoE.kicad_sch (KiCad schematic)
At the start: 82 parts, among them J2 ARJM11C7-114-BA-EW2, T1 FA2805, U10 USBLC6-2SC6, U11 USBLC6-2SC6, U3 W5100S, U4 TLV431DBZ, U5 VO618A, U6 SI3402, U8 VO618A, Y2 25MHz

Commit message: Routing half done
Connections:
- net GND: now also U3.49 (GND)
Changed lines of the file:
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@@
     (pin "47")
     (pin "48")
+    (pin "49")
     (pin "5")
     (pin "6")
