File: _autosave-repeat-hw.kicad_sch (KiCad schematic)
At the start: 75 parts, among them J1 USB_C_Receptacle_USB2.0, J3 ANT2, J4 Programming header, U1 nRF5340-QKxx, U12 MX25R3235FZNxx0, U2 USBLC6-2SC6, U7 nRF21540, U9 AMS1117-3.3, Y1 32MHz

Commit message: Routing almost done
Parts:
- gave numbers to parts that had none: 1
Changed lines of the file:
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@@
   (symbol (lib_id "Device:C") (at 220.98 36.83 0) (unit 1)
     (in_bom yes) (on_board yes) (fields_autoplaced)
-    (property "Reference" "C?" (id 0) (at 224.79 35.5599 0)
+    (property "Reference" "C58" (id 0) (at 224.79 35.5599 0)
       (effects (font (size 1.27 1.27)) (justify left))
     )
@@
       (reference "C57") (unit 1) (value "10u") (footprint "Capacitor_SMD:C_0603_1608Metric")
     )
+    (path "/b2cdb508-e037-4325-8bd7-acc30cde1a17"
+      (reference "C58") (unit 1) (value "10u") (footprint "Capacitor_SMD:C_0603_1608Metric")
+    )
     (path "/01a0d8c5-859a-4d96-9336-4d8c0caf02dd/2d2d6887-f213-4625-89f7-11677df2f36b"
       (reference "C59") (unit 1) (value "1u") (footprint "Capacitor_SMD:C_0603_1608Metric")
@@
       (reference "C84") (unit 1) (value "100n") (footprint "Capacitor_SMD:C_0402_1005Metric")
     )
-    (path "/b2cdb508-e037-4325-8bd7-acc30cde1a17"
-      (reference "C?") (unit 1) (value "10u") (footprint "Capacitor_SMD:C_0603_1608Metric")
-    )
     (path "/9fc025c2-ef9d-4875-8369-89248e04bab7"
