File: repeat-hw.kicad_sch (KiCad schematic)
At the start: 75 parts, among them J1 USB_C_Receptacle_USB2.0, J3 ANT2, J4 Programming header, U1 nRF5340-QKxx, U12 MX25R3235FZNxx0, U2 USBLC6-2SC6, U7 nRF21540, U9 AMS1117-3.3, Y1 32MHz

Commit message: Routing done
Parts:
- removed AE2: NFC, symbol Device:Antenna_Loop
- added TP3, TP4: TestPoint, TestPoint:TestPoint_Pad_D1.0mm, symbol Connector:TestPoint
- gave numbers to parts that had none: 1
Connections:
- net NFC1: now also TP3.1
- net NFC2: now also TP4.1
- net PLOSS: now also U1.B24 (P0.30)
- no-connect marks 32 -> 31
Changed lines of the file:
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@@
   (no_connect (at 359.41 160.02))
   (no_connect (at 262.89 128.27))
-  (no_connect (at 262.89 201.93))
   (no_connect (at 262.89 156.21))
   (no_connect (at 49.53 115.57))
@@
     (stroke (width 0) (type default) (color 0 0 0 0))
   )
+  (wire (pts (xy 262.89 201.93) (xy 275.59 201.93))
+    (stroke (width 0) (type default) (color 0 0 0 0))
+  )
   (wire (pts (xy 355.6 195.58) (xy 355.6 196.85))
     (stroke (width 0) (type default) (color 0 0 0 0))
@@
     (effects (font (size 1.27 1.27)) (justify right bottom))
   )
+  (label "PLOSS" (at 275.59 201.93 180)
+    (effects (font (size 1.27 1.27)) (justify right bottom))
+  )
   (label "USENSE_USB" (at 275.59 135.89 180)
     (effects (font (size 1.27 1.27)) (justify right bottom))
@@
     (pin "1")
   )
-  (symbol (lib_id "Device:Antenna_Loop") (at 312.42 130.81 270) (unit 1)
+  (symbol (lib_id "Connector:TestPoint") (at 307.34 130.81 270) (unit 1)
     (in_bom yes) (on_board yes) (fields_autoplaced)
-    (property "Reference" "AE2" (id 0) (at 317.5 130.8099 90)
+    (property "Reference" "TP3" (id 0) (at 312.42 130.8099 90)
       (effects (font (size 1.27 1.27)) (justify left))
     )
-    (property "Value" "NFC" (id 1) (at 317.5 133.3499 90)
-      (effects (font (size 1.27 1.27)) (justify left))
+    (property "Value" "TestPoint" (id 1) (at 312.42 132.0799 90)
+      (effects (font (size 1.27 1.27)) (justify left) hide)
     )
-    (property "Footprint" "" (id 2) (at 312.42 130.81 0)
+    (property "Footprint" "TestPoint:TestPoint_Pad_D1.0mm" (id 2) (at 307.34 135.89 0)
       (effects (font (size 1.27 1.27)) hide)
     )
-    (property "Datasheet" "~" (id 3) (at 312.42 130.81 0)
+    (property "Datasheet" "~" (id 3) (at 307.34 135.89 0)
       (effects (font (size 1.27 1.27)) hide)
     )
     (pin "1")
-    (pin "2")
   )
   (symbol (lib_id "power:+3V3") (at 153.67 58.42 0) (mirror y) (unit 1)
@@
   (symbol (lib_id "Device:C") (at 220.98 36.83 0) (unit 1)
     (in_bom yes) (on_board yes) (fields_autoplaced)
-    (property "Reference" "C?" (id 0) (at 224.79 35.5599 0)
+    (property "Reference" "C58" (id 0) (at 224.79 35.5599 0)
       (effects (font (size 1.27 1.27)) (justify left))
     )
@@
     (pin "G")
   )
+  (symbol (lib_id "Connector:TestPoint") (at 307.34 133.35 270) (unit 1)
+    (in_bom yes) (on_board yes) (fields_autoplaced)
+    (property "Reference" "TP4" (id 0) (at 312.42 133.3499 90)
+      (effects (font (size 1.27 1.27)) (justify left))
+    )
+    (property "Value" "TestPoint" (id 1) (at 312.42 134.6199 90)
+      (effects (font (size 1.27 1.27)) (justify left) hide)
+    )
+    (property "Footprint" "TestPoint:TestPoint_Pad_D1.0mm" (id 2) (at 307.34 138.43 0)
+      (effects (font (size 1.27 1.27)) hide)
+    )
+    (property "Datasheet" "~" (id 3) (at 307.34 138.43 0)
+      (effects (font (size 1.27 1.27)) hide)
+    )
+    (pin "1")
+  )
   (symbol (lib_id "Device:L") (at 59.69 250.19 90) (unit 1)
     (in_bom yes) (on_board yes) (fields_autoplaced)
@@
       (reference "AE1") (unit 1) (value "SWRA117D") (footprint "RF_Antenna:Texas_SWRA117D_2.4GHz_Right")
     )
-    (path "/78f18a00-49f5-4cf2-8147-a2f01d81a80a"
-      (reference "AE2") (unit 1) (value "NFC") (footprint "")
-    )
     (path "/fd889ac9-1962-456d-88ed-02084d2b0adc"
       (reference "C1") (unit 1) (value "4u7") (footprint "Capacitor_SMD:C_0603_1608Metric")
@@
       (reference "C57") (unit 1) (value "10u") (footprint "Capacitor_SMD:C_0603_1608Metric")
     )
+    (path "/b2cdb508-e037-4325-8bd7-acc30cde1a17"
+      (reference "C58") (unit 1) (value "10u") (footprint "Capacitor_SMD:C_0603_1608Metric")
+    )
     (path "/01a0d8c5-859a-4d96-9336-4d8c0caf02dd/2d2d6887-f213-4625-89f7-11677df2f36b"
       (reference "C59") (unit 1) (value "1u") (footprint "Capacitor_SMD:C_0603_1608Metric")
@@
       (reference "C84") (unit 1) (value "100n") (footprint "Capacitor_SMD:C_0402_1005Metric")
     )
-    (path "/b2cdb508-e037-4325-8bd7-acc30cde1a17"
-      (reference "C?") (unit 1) (value "10u") (footprint "Capacitor_SMD:C_0603_1608Metric")
-    )
     (path "/9fc025c2-ef9d-4875-8369-89248e04bab7"
       (reference "D1") (unit 1) (value "BAV99") (footprint "Package_TO_SOT_SMD:SOT-23")
@@
       (reference "TP2") (unit 1) (value "MM8130-2600") (footprint "murrata:MM8130-2600")
     )
+    (path "/83f75ee7-0a6c-4734-a238-547f38a837a8"
+      (reference "TP3") (unit 1) (value "TestPoint") (footprint "TestPoint:TestPoint_Pad_D1.0mm")
+    )
+    (path "/ce14917c-b6a4-4595-b392-fbf962c3915a"
+      (reference "TP4") (unit 1) (value "TestPoint") (footprint "TestPoint:TestPoint_Pad_D1.0mm")
+    )
     (path "/eef2ffeb-713f-4ed1-ad4d-f8ab8bfc27bc"
